File: Omega2 mini-dock.kicad_pcb (KiCad board)
At the start: 2 copper layers, 38.1 x 61 mm, 16 parts, among them P1 USB_OTG, P2 USB_A, P3 CONN_01X16, P5 CONN_01X16, U1 LM1117-3.3, U2 Omega2

Commit message: Some tuning on the visuals
Parts:
- removed POWER: CONN_02X04, Pin_Headers:Pin_Header_Straight_2x04_Pitch2.54mm
- added G***: LOGO, omega2:WereCatf-logo, B.Cu at (124.5, 115.6)
- added POWER_HDR1: CONN_02X04, Pin_Headers:Pin_Header_Straight_2x04_Pitch2.54mm, F.Cu at (139.7, 81.3)
